File: KiCad/PicVision.sch (KiCad schematic (older format))
At the start: 40 parts, among them CON1 Power input, J1 video out, J2 audio_out, P1 ICSP, P2 SPI2, P3 I2C 2, P4 PAL VIDEO, P5 gamepad 1, P6 gamepad 2, SW1 SPST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

Commit message: stripboard wiring
Parts:
- removed P5: gamepad 1, symbol CONN_7
- removed P6: gamepad 2, symbol CONN_7
- added P5, P6: gamepad 2, symbol CONN_5
- gave numbers to parts that had none: 1
Connections:
- wire segments 114 -> 113
Other:
- moved on the sheet: F1, SW1
Changed lines of the file:
@@
 LIBS:contrib
 LIBS:valves
+LIBS:librairie-personnelle
 LIBS:PicVision-cache
 EELAYER 27 0
@@
 Sheet 1 1
 Title ""
-Date "4 mar 2014"
+Date "8 mar 2014"
 Rev ""
 Comp ""
@@
 F 3 "" H 6800 4700 60  0000 C CNN
 	1    6800 4700
-	1    0    0    -1
-$EndComp
-$Comp
-L CONN_7 P5
-U 1 1 530CCABD
-P 8400 1300
-F 0 "P5" V 8370 1300 60  0000 C CNN
-F 1 "gamepad 1" V 8470 1300 60  0000 C CNN
-F 2 "" H 8400 1300 60  0000 C CNN
-F 3 "" H 8400 1300 60  0000 C CNN
-	1    8400 1300
-	1    0    0    -1
-$EndComp
-$Comp
-L CONN_7 P6
-U 1 1 530CCACA
-P 8400 2200
-F 0 "P6" V 8370 2200 60  0000 C CNN
-F 1 "gamepad 2" V 8470 2200 60  0000 C CNN
-F 2 "" H 8400 2200 60  0000 C CNN
-F 3 "" H 8400 2200 60  0000 C CNN
-	1    8400 2200
 	1    0    0    -1
 $EndComp
@@
 L SPST SW1
 U 1 1 530CFF0A
-P 3150 6100
-F 0 "SW1" H 3150 6200 39  0000 C CNN
-F 1 "SPST" H 3150 6000 70  0000 C CNN
-F 2 "" H 3150 6100 60  0000 C CNN
-F 3 "" H 3150 6100 60  0000 C CNN
-	1    3150 6100
+P 2500 6100
+F 0 "SW1" H 2500 6200 39  0000 C CNN
+F 1 "SPST" H 2500 6000 70  0000 C CNN
+F 2 "" H 2500 6100 60  0000 C CNN
+F 3 "" H 2500 6100 60  0000 C CNN
+	1    2500 6100
 	1    0    0    -1
 $EndComp
@@
 L FUSE F1
 U 1 1 530FBA17
-P 2250 6100
-F 0 "F1" H 2350 6150 40  0000 C CNN
-F 1 "500mA" H 2150 6050 40  0000 C CNN
-F 2 "~" H 2250 6100 60  0000 C CNN
-F 3 "~" H 2250 6100 60  0000 C CNN
-	1    2250 6100
+P 3400 6100
+F 0 "F1" H 3500 6150 40  0000 C CNN
+F 1 "500mA" H 3300 6050 40  0000 C CNN
+F 2 "~" H 3400 6100 60  0000 C CNN
+F 3 "~" H 3400 6100 60  0000 C CNN
+	1    3400 6100
 	1    0    0    -1
 $EndComp
@@
 	8200 5050 8200 5250
 Wire Wire Line
-	8050 1600 8050 1700
-Wire Wire Line
-	8050 2500 8050 2600
+	8050 1400 8050 1700
+Wire Wire Line
+	8050 2300 8050 2600
 Wire Wire Line
 	7850 1900 8050 1900
@@
 Wire Wire Line
 	7850 2200 8050 2200
-Wire Wire Line
-	7850 2300 8050 2300
 Wire Wire Line
 	8200 6000 8200 6250
@@
 Wire Wire Line
 	7700 3700 7700 3800
-Wire Wire Line
-	2500 6100 2650 6100
 Wire Wire Line
 	7600 2700 7600 3000
@@
 NOISE
 $Comp
-L R R?
+L R R12
 U 1 1 5314EEB5
 P 7050 5300
-F 0 "R?" V 7130 5300 40  0000 C CNN
+F 0 "R12" V 7130 5300 40  0000 C CNN
 F 1 "10K" V 7057 5301 40  0000 C CNN
 F 2 "~" V 6980 5300 30  0000 C CNN
@@
 	7300 5300 7350 5300
 Connection ~ 7350 5650
+$Comp
+L CONN_5 P6
+U 1 1 531B74FB
+P 8450 2100
+F 0 "P6" V 8400 2100 50  0000 C CNN
+F 1 "gamepad 2" V 8500 2100 50  0000 C CNN
+F 2 "" H 8450 2100 60  0000 C CNN
+F 3 "" H 8450 2100 60  0000 C CNN
+	1    8450 2100
+	1    0    0    -1
+$EndComp
+$Comp
+L CONN_5 P5
+U 1 1 531B759B
+P 8450 1200
+F 0 "P5" V 8400 1200 50  0000 C CNN
+F 1 "gamepad 2" V 8500 1200 50  0000 C CNN
+F 2 "" H 8450 1200 60  0000 C CNN
+F 3 "" H 8450 1200 60  0000 C CNN
+	1    8450 1200
+	1    0    0    -1
+$EndComp
+Wire Wire Line
+	3000 6100 3150 6100
 $EndSCHEMATC

Commit message: mod. to electronic schematic
Parts:
- added CON?: SNES, symbol SNES
- R4: value R -> 150R
Other:
- note added: "SNES controler\nconnector"
Changed lines of the file:
@@
 Sheet 1 1
 Title ""
-Date "8 mar 2014"
+Date "10 mar 2014"
 Rev ""
 Comp ""
@@
 P 4750 6550
 F 0 "R4" V 4830 6550 50  0000 C CNN
-F 1 "R" V 4750 6550 50  0000 C CNN
+F 1 "150R" V 4750 6550 50  0000 C CNN
 F 2 "" H 4750 6550 60  0000 C CNN
 F 3 "" H 4750 6550 60  0000 C CNN
@@
 Wire Wire Line
 	3000 6100 3150 6100
+$Comp
+L SNES CON?
+U 1 1 531DB6C0
+P 9700 1800
+F 0 "CON?" H 9700 1400 60  0000 C CNN
+F 1 "SNES" H 9650 2400 60  0000 C CNN
+F 2 "" H 9700 1800 60  0000 C CNN
+F 3 "" H 9700 1800 60  0000 C CNN
+	1    9700 1800
+	1    0    0    -1
+$EndComp
+Text Notes 9450 1050 0    60   ~ 0
+SNES controler\nconnector
 $EndSCHEMATC

Commit message: mod. to electronic schemtatic
Other:
- note added: "SNES controller\nconnector"
- note removed: "SNES controler\nconnector"
Changed lines of the file:
@@
 $EndComp
 Text Notes 9450 1050 0    60   ~ 0
-SNES controler\nconnector
+SNES controller\nconnector
 $EndSCHEMATC

Commit message: added assembly photos
Parts:
- added C12: 2n2, symbol C
- C7: value 4n7 -> 2n2
- R4: value 150R -> 200R
- U1: value UA78M33 -> L78L33
- gave numbers to parts that had none: 1
Connections:
- net GND: now also C12.2
- net at C7.1, R6.2, R7.1: now also C12.1
Changed lines of the file:
@@
 Sheet 1 1
 Title ""
-Date "10 mar 2014"
+Date "12 mar 2014"
 Rev ""
 Comp ""
@@
 P 4150 6300
 F 0 "U1" H 4150 6600 60  0000 C CNN
-F 1 "UA78M33" H 4150 6500 60  0000 C CNN
+F 1 "L78L33" H 4150 6500 60  0000 C CNN
 F 2 "~" H 4150 6300 60  0000 C CNN
 F 3 "~" H 4150 6300 60  0000 C CNN
@@
 P 4750 6550
 F 0 "R4" V 4830 6550 50  0000 C CNN
-F 1 "150R" V 4750 6550 50  0000 C CNN
+F 1 "200R" V 4750 6550 50  0000 C CNN
 F 2 "" H 4750 6550 60  0000 C CNN
 F 3 "" H 4750 6550 60  0000 C CNN
@@
 P 6700 5950
 F 0 "C7" H 6750 6050 50  0000 L CNN
-F 1 "4n7" H 6750 5850 50  0000 L CNN
+F 1 "2n2" H 6750 5850 50  0000 L CNN
 F 2 "" H 6700 5950 60  0000 C CNN
 F 3 "" H 6700 5950 60  0000 C CNN
@@
 	3000 6100 3150 6100
 $Comp
-L SNES CON?
+L SNES CON2
 U 1 1 531DB6C0
 P 9700 1800
-F 0 "CON?" H 9700 1400 60  0000 C CNN
+F 0 "CON2" H 9700 1400 60  0000 C CNN
 F 1 "SNES" H 9650 2400 60  0000 C CNN
 F 2 "" H 9700 1800 60  0000 C CNN
@@
 Text Notes 9450 1050 0    60   ~ 0
 SNES controller\nconnector
+$Comp
+L C C12
+U 1 1 5320955C
+P 6350 5950
+F 0 "C12" H 6400 6050 50  0000 L CNN
+F 1 "2n2" H 6400 5850 50  0000 L CNN
+F 2 "" H 6350 5950 60  0000 C CNN
+F 3 "" H 6350 5950 60  0000 C CNN
+	1    6350 5950
+	1    0    0    -1
+$EndComp
+Wire Wire Line
+	6700 6150 6350 6150
+Wire Wire Line
+	6700 5750 6350 5750
 $EndSCHEMATC

Commit message: schematic update + bom
Parts:
- R4: value 200R -> 75R
Changed lines of the file:
@@
 Sheet 1 1
 Title ""
-Date "12 mar 2014"
+Date "14 mar 2014"
 Rev ""
 Comp ""
@@
 P 4750 6550
 F 0 "R4" V 4830 6550 50  0000 C CNN
-F 1 "200R" V 4750 6550 50  0000 C CNN
+F 1 "75R" V 4750 6550 50  0000 C CNN
 F 2 "" H 4750 6550 60  0000 C CNN
 F 3 "" H 4750 6550 60  0000 C CNN

Commit message: schematic update
Parts:
- D1: value Power LED -> Power indicator
Other:
- note added: "RED LED"
Changed lines of the file:
@@
 P 4750 7050
 F 0 "D1" H 4750 7150 50  0000 C CNN
-F 1 "Power LED" V 4750 6750 50  0000 C CNN
+F 1 "Power indicator" V 4750 6700 50  0000 C CNN
 F 2 "" H 4750 7050 60  0000 C CNN
 F 3 "" H 4750 7050 60  0000 C CNN
@@
 Wire Wire Line
 	6700 5750 6350 5750
+Text Notes 4900 7100 0    60   ~ 0
+RED LED
 $EndSCHEMATC
